File: puenteH/puenteH.kicad_pcb (KiCad board)
At the start: 2 copper layers, 138.6 x 160 mm, 51 parts, among them J1 Conn_01x02, J2 Conn_01x02, J3 Conn_01x02, J4 Conn_01x02, J5 Conn_01x02, Q1 TIP127, Q10 TIP127, Q11 TIP122, Q12 TIP122, Q13 TIP122, Q14 TIP127, Q15 TIP122, Q16 TIP127, Q17 TIP122, Q18 TIP122, Q2 TIP127, Q3 TIP122, Q4 TIP122, Q5 TIP122, Q6 TIP122, Q7 TIP122, Q8 TIP127, Q9 TIP122, U1 LM7805_TO220

Commit message: Schematic and PCB design finished
Parts:
- removed C1, C2: C, Capacitor_THT:C_Disc_D4.7mm_W2.5mm_P5.00mm
- removed the J2 at (158.0, 39.5)
- removed U1: LM7805_TO220, Package_TO_SOT_THT:TO-220-3_Horizontal_TabDown
- added REF**: KiCad-Logo_12mm_SilkScreen, Symbol:KiCad-Logo_12mm_SilkScreen, F.Cu at (172.0, 155.7)
- added REF**: OSHW-Logo_19x20mm_SilkScreen, Symbol:OSHW-Logo_19x20mm_SilkScreen, F.Cu at (92.5, 103.0)
- renumbered J3 to J2, J4 to J3, J5 to J4
Routing:
- net Net-(J2-Pin_1): track 123.4 -> 0.00 mm
- net Net-(D10-A): track 314.7 -> 241.8 mm
- net Net-(D1-K): track 274.4 -> 242.3 mm, vias 0 -> 1
- net Net-(Q13-B): track 102.5 -> 109.2 mm, vias 1 -> 2
- net Net-(Q18-B): track 101.5 -> 106.1 mm, vias 3 -> 0
- net Net-(Q12-B): track 70.8 -> 71.9 mm
Other:
- outline, holes or cut-outs redrawn
- board text added: "https://github.com/ian16munoz3nunez1/hueSort.git"
