File: puenteH/puenteH.kicad_sch (KiCad schematic)
At the start: 51 parts, among them J1 Conn_01x02, J2 Conn_01x02, J3 Conn_01x02, J4 Conn_01x02, J5 Conn_01x02, J6 Conn_01x06, Q1 TIP127, Q10 TIP127, Q11 TIP122, Q12 TIP122, Q13 TIP122, Q14 TIP127, Q15 TIP122, Q16 TIP127, Q17 TIP122, Q18 TIP122, Q2 TIP127, Q3 TIP122, Q4 TIP122, Q5 TIP122, Q6 TIP122, Q7 TIP122, Q8 TIP127, Q9 TIP122, U1 LM7805_TO220

Commit message: Schematic and PCB design finished
Parts:
- removed C1, C2: C, Capacitor_THT:C_Disc_D4.7mm_W2.5mm_P5.00mm, symbol Device:C
- removed J2: Conn_01x02, TerminalBlock:TerminalBlock_bornier-2_P5.08mm, symbol Connector_Generic:Conn_01x02
- removed U1: LM7805_TO220, Package_TO_SOT_THT:TO-220-3_Horizontal_TabDown, symbol Regulator_Linear:LM7805_TO220
- renumbered J3 to J2, J4 to J3, J5 to J4
